File: led_dimmer.sch (KiCad schematic (older format))
At the start: 13 parts, among them P1 CONN_2, P2 CONN_2, Q1 MOSFET_N, U1 555

Commit message: tweaks
Parts:
- Q1: value MOSFET_N -> TSM2314CX
Changed lines of the file:
@@
 LIBS:valves
 LIBS:ds_device
+LIBS:led_dimmer-cache
 EELAYER 24 0
 EELAYER END
@@
 P 7100 3300
 F 0 "Q1" H 7110 3470 60  0000 R CNN
-F 1 "MOSFET_N" H 7110 3150 60  0000 R CNN
+F 1 "TSM2314CX" H 7110 3150 60  0000 R CNN
 F 2 "" H 7100 3300 60  0000 C CNN
 F 3 "" H 7100 3300 60  0000 C CNN
